File: node.sch (KiCad schematic (older format))
At the start: 16 parts, among them J1 Conn_01x04_Male, J2 Conn_01x04_Male, J3 USB_B_Mini, J4 Conn_02x05_Odd_Even, SW1 SW_Push, SW2 SW_Push, U1 AMS1117-3.3, U2 USBLC6-2SC6, U3 CDSENET_E22-900M22S, U4 STM32L083VBTx

Commit message: hello
Parts:
- removed J1, J2: Conn_01x04_Male, Connectors_JST:JST_PH_S4B-PH-K_04x2.00mm_Angled, symbol Connector:Conn_01x04_Male
- added J4P1, J4P2: Conn_01x04, symbol Connector_Generic:Conn_01x04
- added J6P3: Conn_01x06, symbol Connector_Generic:Conn_01x06
- U2: symbol Power_Protection:USBLC6-2SC6 -> node-rescue:USBLC6-2SC6-Power_Protection
- U3: symbol LoRa:CDSENET_E22-900M22S -> node-rescue:CDSENET_E22-900M22S-LoRa
- renumbered J4 to J10STLINK, SW2 to SW_BOOT0, SW1 to SW_NRST
Connections:
- net labels added: SWIM
- net labels removed: SWO
- wire segments 91 -> 83
- no-connect marks 2 -> 0
Other:
- moved on the sheet: C1, R1, SW_BOOT0, SW_NRST
